Commit message: Optimize 3 waypoints, openCV and nav2 and complete person detection

File: src/patrol_robot_description/urdf/patrol_robot.urdf (robot description, URDF)
Before this commit: robot sensor_robot, 7 links, 6 joints
Joints:
- joint camera_joint: origin xyz=0.16 0 0.06 rpy=0 0 0 -> xyz=0.16 0 0.30 rpy=0 0 0
